Commit message: fixed issue with transforms; seperated sim and real robot urdf; updated nav2 params

File: sim_ws/src/glide_robot/models/glide_description.urdf.xacro (robot description, xacro)
@@ -138,5 +138,5 @@
     <visual>
       <geometry>
-        <box size="${body_length} ${body_width} ${body_height}"/>
+        <box size="${body_width} ${body_length} ${body_height}"/>
       </geometry>
       <origin rpy="0 0 1.57" xyz="0 0 ${body_center}"/>
@@ -242,5 +242,5 @@
   </link>
   <joint name="base_to_human" type="fixed">
-    <origin rpy="0 ${degrees_90} 0" xyz="0.0 -1.0 ${2*wheel_radius}"/>
+    <origin rpy="0 ${degrees_90} 0" xyz="-1.0 0.0 ${2*wheel_radius}"/>
     <parent link="base_link"/>
     <child link="human_link"/>

File: sim_ws/src/glide_robot/models/sim_glide_description.urdf (robot description, URDF)
Before this commit: robot glide, 7 links, 6 joints
Links:
- removed link base_footprint
- added link camera_color_frame
- added link camera_color_optical_frame
- added link camera_depth_frame
- added link camera_depth_optical_frame
- added link camera_left_ir_frame
- added link camera_left_ir_optical_frame
- added link camera_link
- added link camera_right_ir_frame
- added link camera_right_ir_optical_frame
- link base_link: geometry visual box size=0.3 0.2 0.1
Joints:
- removed joint base_joint
- added joint camera_color_joint: type fixed, parent camera_depth_frame, child camera_color_frame
- added joint camera_color_optical_joint: type fixed, parent camera_color_frame, child camera_color_optical_frame
- added joint camera_depth_joint: type fixed, parent camera_link, child camera_depth_frame
- added joint camera_depth_optical_joint: type fixed, parent camera_depth_frame, child camera_depth_optical_frame
- added joint camera_left_ir_joint: type fixed, parent camera_depth_frame, child camera_left_ir_frame
- added joint camera_left_ir_optical_joint: type fixed, parent camera_left_ir_frame, child camera_left_ir_optical_frame
- added joint camera_link_joint: type fixed, parent base_link, child camera_link
- added joint camera_right_ir_joint: type fixed, parent camera_depth_frame, child camera_right_ir_frame
- added joint camera_right_ir_optical_joint: type fixed, parent camera_right_ir_frame, child camera_right_ir_optical_frame
- joint front_left_wheel_joint: origin xyz=0.13175 -0.061900000000000004 0.107 rpy=0 0 3.141592653589793 -> xyz=-0.061900000000000004 0.13175 0.077 rpy=1.5707963267948966 0 3.141592653589793
- joint front_right_wheel_joint: origin xyz=-0.13175 -0.061900000000000004 0.107 rpy=0 0 3.141592653589793 -> xyz=-0.061900000000000004 -0.13175 0.077 rpy=1.5707963267948966 0 3.141592653589793
- joint rear_left_wheel_joint: origin xyz=0 0 0 rpy=1.5707963267948966 0 3.141592653589793 -> xyz=-1.0 0.13175 0.077 rpy=1.5707963267948966 0 3.141592653589793
- joint rear_right_wheel_joint: origin xyz=0 0 0 rpy=1.5707963267948966 0 3.141592653589793 -> xyz=-1.0 -0.13175 0.077 rpy=1.5707963267948966 0 3.141592653589793

File: sim_ws/src/glide_robot/models/sim_glide_description.urdf.xacro (robot description, xacro)
@@ -75,5 +75,5 @@
     <joint name="front_${name}_wheel_joint" type="revolute">
       <limit lower="-0.6" upper="0.6" effort="100" velocity="1"/>
-      <origin rpy="${degrees_90} 0 ${pi}" xyz="${offset + wheel_offset} ${xy_reflect * (wheel_gap + body_width/2)} ${wheel_radius + 0.03}"/>
+      <origin rpy="${degrees_90} 0 ${pi}" xyz="${offset + wheel_offset} ${xy_reflect * (wheel_gap + body_width/2)} ${wheel_radius}"/>
       <parent link="base_link"/>
       <child link="front_${name}_wheel"/>
@@ -86,13 +86,13 @@
       <visual>
         <geometry>
-          <cylinder length="0.001" radius="0.001"/>
-        </geometry>
-        <origin rpy="0 0 0" xyz="0 0 0"/>
-        <material name="white"/>
-      </visual>
-      <collision>
-        <origin rpy="0 0 0" xyz="0 0 0"/>
-        <geometry>
-          <cylinder length="0.001" radius="0.001"/>
+          <cylinder length="${wheel_width}" radius="${wheel_radius}"/>
+        </geometry>
+        <origin rpy="0 0 0" xyz="0 0 0"/>
+        <material name="white"/>
+      </visual>
+      <collision>
+        <origin rpy="0 0 0" xyz="0 0 0"/>
+        <geometry>
+          <cylinder length="${wheel_width}" radius="${wheel_radius}"/>
         </geometry>
       </collision>
@@ -106,5 +106,5 @@
     </link>
     <joint name="rear_${name}_wheel_joint" type="continuous">
-      <origin rpy="${degrees_90} 0 ${pi}" xyz="0 0 0"/>
+      <origin rpy="${degrees_90} 0 ${pi}" xyz="-1.0 ${xy_reflect * (wheel_gap + body_width/2)} ${wheel_radius}"/>
       <parent link="base_link"/>
       <child link="rear_${name}_wheel"/>
@@ -134,5 +134,4 @@
       <axis xyz="0 1 0"/>
     </joint> -->
-  <link name="base_footprint"/>
   <link name="base_link">
     <visual>
@@ -147,9 +146,4 @@
       <material>Gazebo/Blue</material>
   </gazebo>
-  <joint name="base_joint" type="fixed">
-      <origin rpy="0 0 0" xyz="0 0 0"/> <!-- 0 3.14 1.57-->
-      <child link="base_link"/>
-      <parent link="base_footprint"/>
-  </joint>
   <!-- <xacro:bar name="front" x_offset="${1.25*body_width}" z_offset="-${body_width}" parent_link="steer_bar_link"/> -->
   <xacro:steer_wheel name="right" offset="-0.1" xy_reflect="-1"/>
