Commit message: fixed sim urdf

File: sim_ws/src/glide_robot/models/sim_glide_description.urdf (robot description, URDF)
Before this commit: robot glide, 15 links, 14 joints
Links:
- added link camera_bottom_screw_frame; collision box size=0.02505 0.090 0.025; visual box size=0.02505 0.090 0.025
Joints:
- added joint camera_joint: type fixed, parent base_link, child camera_bottom_screw_frame
- joint camera_link_joint: parent base_link -> camera_bottom_screw_frame
- joint front_left_wheel_joint: origin xyz=-0.061900000000000004 0.13175 0.077 rpy=1.5707963267948966 0 3.141592653589793 -> xyz=-0.061900000000000004 0.13175 0.107 rpy=1.5707963267948966 0 3.141592653589793
- joint front_right_wheel_joint: origin xyz=-0.061900000000000004 -0.13175 0.077 rpy=1.5707963267948966 0 3.141592653589793 -> xyz=-0.061900000000000004 -0.13175 0.107 rpy=1.5707963267948966 0 3.141592653589793
- joint rear_left_wheel_joint: origin xyz=-1.0 0.13175 0.077 rpy=1.5707963267948966 0 3.141592653589793 -> xyz=0 0 0 rpy=1.5707963267948966 0 3.141592653589793
- joint rear_right_wheel_joint: origin xyz=-1.0 -0.13175 0.077 rpy=1.5707963267948966 0 3.141592653589793 -> xyz=0 0 0 rpy=1.5707963267948966 0 3.141592653589793

File: sim_ws/src/glide_robot/models/sim_glide_description.urdf.xacro (robot description, xacro)
@@ -75,5 +75,5 @@
     <joint name="front_${name}_wheel_joint" type="revolute">
       <limit lower="-0.6" upper="0.6" effort="100" velocity="1"/>
-      <origin rpy="${degrees_90} 0 ${pi}" xyz="${offset + wheel_offset} ${xy_reflect * (wheel_gap + body_width/2)} ${wheel_radius}"/>
+      <origin rpy="${degrees_90} 0 ${pi}" xyz="${offset + wheel_offset} ${xy_reflect * (wheel_gap + body_width/2)} ${wheel_radius + 0.03}"/>
       <parent link="base_link"/>
       <child link="front_${name}_wheel"/>
@@ -106,5 +106,5 @@
     </link>
     <joint name="rear_${name}_wheel_joint" type="continuous">
-      <origin rpy="${degrees_90} 0 ${pi}" xyz="-1.0 ${xy_reflect * (wheel_gap + body_width/2)} ${wheel_radius}"/>
+      <origin rpy="${degrees_90} 0 ${pi}" xyz="0 0 0"/>
       <parent link="base_link"/>
       <child link="rear_${name}_wheel"/>
@@ -156,5 +156,5 @@
   <xacro:rotate_wheel name="right" offset="-0.1" xy_reflect="-1" />
   <xacro:rotate_wheel name="left" offset="-0.1" xy_reflect="1" />
-<!-- <link name="camera_bottom_screw_frame">
+<link name="camera_bottom_screw_frame">
     <visual>
       <geometry>
@@ -167,5 +167,5 @@
       </geometry>
     </collision>
-  </link> -->
+  </link>
   <link name="camera_link"></link>
   <link name="camera_depth_frame"></link>
@@ -177,11 +177,11 @@
   <link name="camera_right_ir_frame"></link>
   <link name="camera_right_ir_optical_frame"></link>
-   <!-- <joint name="camera_joint" type="fixed">
+   <joint name="camera_joint" type="fixed">
     <parent link="base_link" />
     <child link="camera_bottom_screw_frame" />
     <pose xyz="0.4 0 0.25" rpy="0 0 0" />
-  </joint> -->
+  </joint>
   <joint name="camera_link_joint" type="fixed">
-    <parent link="base_link" />
+    <parent link="camera_bottom_screw_frame" />
     <child link="camera_link" />
     <pose xyz="0 0.0175 0.0125 " rpy="0 0 0" />

Commit message: added scripts for generating trajectories from waypoints; updated sim urdf; added new world file

File: sim_ws/src/glide_robot/models/sim_glide_description.urdf (robot description, URDF)
Before this commit: robot glide, 16 links, 15 joints
Joints:
- joint base_to_human: origin xyz=-1.0 0.0 0.154 rpy=0 1.5707963267948966 0 -> xyz=-0.5 0.0 0.2 rpy=0 1.5707963267948966 0
- joint front_left_wheel_joint: limit lower=-0.6 upper=0.6 effort=100 velocity=1 -> lower=-0.9 upper=0.9 effort=100 velocity=1; origin xyz=-0.061900000000000004 0.13175 0.107 rpy=1.5707963267948966 0 3.141592653589793 -> xyz=-0.061900000000000004 0.13175 0.077 rpy=1.5707963267948966 0 3.141592653589793
- joint front_right_wheel_joint: limit lower=-0.6 upper=0.6 effort=100 velocity=1 -> lower=-0.9 upper=0.9 effort=100 velocity=1; origin xyz=-0.061900000000000004 -0.13175 0.107 rpy=1.5707963267948966 0 3.141592653589793 -> xyz=-0.061900000000000004 -0.13175 0.077 rpy=1.5707963267948966 0 3.141592653589793
- joint rear_left_wheel_joint: origin xyz=0 0 0 rpy=1.5707963267948966 0 3.141592653589793 -> xyz=-0.5 0.13175 0.077 rpy=1.5707963267948966 0 3.141592653589793
- joint rear_right_wheel_joint: origin xyz=0 0 0 rpy=1.5707963267948966 0 3.141592653589793 -> xyz=-0.5 -0.13175 0.077 rpy=1.5707963267948966 0 3.141592653589793

File: sim_ws/src/glide_robot/models/sim_glide_description.urdf.xacro (robot description, xacro)
@@ -74,6 +74,6 @@
     </gazebo>
     <joint name="front_${name}_wheel_joint" type="revolute">
-      <limit lower="-0.6" upper="0.6" effort="100" velocity="1"/>
-      <origin rpy="${degrees_90} 0 ${pi}" xyz="${offset + wheel_offset} ${xy_reflect * (wheel_gap + body_width/2)} ${wheel_radius + 0.03}"/>
+      <limit lower="-0.9" upper="0.9" effort="100" velocity="1"/>
+      <origin rpy="${degrees_90} 0 ${pi}" xyz="${offset + wheel_offset} ${xy_reflect * (wheel_gap + body_width/2)} ${wheel_radius}"/>
       <parent link="base_link"/>
       <child link="front_${name}_wheel"/>
@@ -106,5 +106,5 @@
     </link>
     <joint name="rear_${name}_wheel_joint" type="continuous">
-      <origin rpy="${degrees_90} 0 ${pi}" xyz="0 0 0"/>
+      <origin rpy="${degrees_90} 0 ${pi}" xyz="-0.5 ${xy_reflect * (wheel_gap + body_width/2)} ${wheel_radius}"/>
       <parent link="base_link"/>
       <child link="rear_${name}_wheel"/>
@@ -236,5 +236,5 @@
   </link>
   <joint name="base_to_human" type="fixed">
-    <origin rpy="0 ${degrees_90} 0" xyz="-1.0 0.0 ${2*wheel_radius}"/>
+    <origin rpy="0 ${degrees_90} 0" xyz="-0.5 0.0 ${2*body_center}"/>
     <parent link="base_link"/>
     <child link="human_link"/>
