Commit message: updated URDF and nav2 parameters; added more submodule dependencies

File: sim_ws/src/glide_robot/models/glide_description.urdf (robot description, URDF)
Before this commit: robot glide, 16 links, 15 joints
Links:
- removed link camera_bottom_screw_frame
- added link base_footprint; visual box size=0.3 0.2 0.1
- link base_link: geometry 
Joints:
- removed joint camera_joint
- added joint base_joint: type fixed, parent base_link, child base_footprint, origin xyz=0 0 0 rpy=0 3.14 1.57
- joint camera_link_joint: parent camera_bottom_screw_frame -> base_link
- joint front_left_wheel_joint: limit lower=-0.9 upper=0.9 effort=100 velocity=1 -> lower=-0.6 upper=0.6 effort=100 velocity=1
- joint front_right_wheel_joint: limit lower=-0.9 upper=0.9 effort=100 velocity=1 -> lower=-0.6 upper=0.6 effort=100 velocity=1

File: sim_ws/src/glide_robot/models/glide_description.urdf.xacro (robot description, xacro)
@@ -134,5 +134,6 @@
       <axis xyz="0 1 0"/>
     </joint> -->
-  <link name="base_link">
+  <link name="base_link"/>
+  <link name="base_footprint">
     <visual>
       <geometry>
@@ -146,4 +147,9 @@
       <material>Gazebo/Blue</material>
   </gazebo>
+  <joint name="base_joint" type="fixed">
+      <origin rpy="0 3.14 1.57" xyz="0 0 0"/>
+      <parent link="base_link"/>
+      <child link="base_footprint"/>
+  </joint>
   <!-- <xacro:bar name="front" x_offset="${1.25*body_width}" z_offset="-${body_width}" parent_link="steer_bar_link"/> -->
   <xacro:steer_wheel name="right" offset="-0.1" xy_reflect="-1"/>
@@ -156,5 +162,5 @@
   <xacro:rotate_wheel name="right" offset="-0.1" xy_reflect="-1" />
   <xacro:rotate_wheel name="left" offset="-0.1" xy_reflect="1" />
-<link name="camera_bottom_screw_frame">
+<!-- <link name="camera_bottom_screw_frame">
     <visual>
       <geometry>
@@ -167,5 +173,5 @@
       </geometry>
     </collision>
-  </link>
+  </link> -->
   <link name="camera_link"></link>
   <link name="camera_depth_frame"></link>
@@ -177,11 +183,11 @@
   <link name="camera_right_ir_frame"></link>
   <link name="camera_right_ir_optical_frame"></link>
-   <joint name="camera_joint" type="fixed">
+   <!-- <joint name="camera_joint" type="fixed">
     <parent link="base_link" />
     <child link="camera_bottom_screw_frame" />
     <pose xyz="0.4 0 0.25" rpy="0 0 0" />
-  </joint>
+  </joint> -->
   <joint name="camera_link_joint" type="fixed">
-    <parent link="camera_bottom_screw_frame" />
+    <parent link="base_link" />
     <child link="camera_link" />
     <pose xyz="0 0.0175 0.0125 " rpy="0 0 0" />

Commit message: Updated urdfs; created separate sim and real urdf

File: sim_ws/src/glide_robot/models/glide_description.urdf (robot description, URDF)
Before this commit: robot glide, 16 links, 15 joints
Links:
- removed link camera_color_frame
- removed link camera_color_optical_frame
- removed link camera_depth_frame
- removed link camera_depth_optical_frame
- removed link camera_left_ir_frame
- removed link camera_left_ir_optical_frame
- removed link camera_link
- removed link camera_right_ir_frame
- removed link camera_right_ir_optical_frame
- link base_footprint: geometry 
- link base_link: geometry visual box size=0.3 0.2 0.1
- link rear_left_wheel: geometry collision cylinder length=0.003 radius=0.077; visual cylinder length=0.003 radius=0.077
- link rear_right_wheel: geometry collision cylinder length=0.003 radius=0.077; visual cylinder length=0.003 radius=0.077
Joints:
- removed joint camera_color_joint
- removed joint camera_color_optical_joint
- removed joint camera_depth_joint
- removed joint camera_depth_optical_joint
- removed joint camera_left_ir_joint
- removed joint camera_left_ir_optical_joint
- removed joint camera_link_joint
- removed joint camera_right_ir_joint
- removed joint camera_right_ir_optical_joint
- joint base_joint: child base_footprint -> base_link; origin xyz=0 0 0 rpy=0 3.14 1.57 -> xyz=0 0 0 rpy=0 0 0; parent base_link -> base_footprint
- joint base_to_human: origin xyz=-1.0 0.0 0.154 rpy=0 1.5707963267948966 0 -> xyz=0.0 -1.0 0.154 rpy=0 1.5707963267948966 0

File: sim_ws/src/glide_robot/sim_glide_description.urdf.xacro (robot description, xacro)
@@ -86,13 +86,13 @@
       <visual>
         <geometry>
-          <cylinder length="${wheel_width}" radius="${wheel_radius}"/>
-        </geometry>
-        <origin rpy="0 0 0" xyz="0 0 0"/>
-        <material name="white"/>
-      </visual>
-      <collision>
-        <origin rpy="0 0 0" xyz="0 0 0"/>
-        <geometry>
-          <cylinder length="${wheel_width}" radius="${wheel_radius}"/>
+          <cylinder length="0.001" radius="0.001"/>
+        </geometry>
+        <origin rpy="0 0 0" xyz="0 0 0"/>
+        <material name="white"/>
+      </visual>
+      <collision>
+        <origin rpy="0 0 0" xyz="0 0 0"/>
+        <geometry>
+          <cylinder length="0.001" radius="0.001"/>
         </geometry>
       </collision>
@@ -140,5 +140,5 @@
         <box size="${body_length} ${body_width} ${body_height}"/>
       </geometry>
-      <origin rpy="0 0 1.57" xyz="0 0 ${body_center}"/>
+      <origin rpy="0 0 0" xyz="0 0 ${body_center}"/>
       <material name="blue"/>
     </visual>
@@ -174,5 +174,5 @@
     </collision>
   </link> -->
-  <!-- <link name="camera_link"></link>
+  <link name="camera_link"></link>
   <link name="camera_depth_frame"></link>
   <link name="camera_depth_optical_frame"></link>
@@ -182,5 +182,5 @@
   <link name="camera_left_ir_optical_frame"></link>
   <link name="camera_right_ir_frame"></link>
-  <link name="camera_right_ir_optical_frame"></link> -->
+  <link name="camera_right_ir_optical_frame"></link>
    <!-- <joint name="camera_joint" type="fixed">
     <parent link="base_link" />
@@ -188,5 +188,5 @@
     <pose xyz="0.4 0 0.25" rpy="0 0 0" />
   </joint> -->
-  <!-- <joint name="camera_link_joint" type="fixed">
+  <joint name="camera_link_joint" type="fixed">
     <parent link="base_link" />
     <child link="camera_link" />
@@ -232,5 +232,5 @@
     <child link="camera_right_ir_optical_frame" />
     <pose xyz="0 0 0 " rpy="-1.57 0 -1.57" />
-  </joint> -->
+  </joint>
   <link name="human_link">
     <visual>
@@ -242,5 +242,5 @@
   </link>
   <joint name="base_to_human" type="fixed">
-    <origin rpy="0 ${degrees_90} 0" xyz="0.0 -1.0 ${2*wheel_radius}"/>
+    <origin rpy="0 ${degrees_90} 0" xyz="-1.0 0.0 ${2*wheel_radius}"/>
     <parent link="base_link"/>
     <child link="human_link"/>

Commit message: reverted glide urdf

File: sim_ws/src/glide_robot/models/glide_description.urdf (robot description, URDF)
Before this commit: robot glide, 16 links, 15 joints
Links:
- removed link camera_bottom_screw_frame
- removed link camera_color_frame
- removed link camera_color_optical_frame
- removed link camera_depth_frame
- removed link camera_depth_optical_frame
- removed link camera_left_ir_frame
- removed link camera_left_ir_optical_frame
- removed link camera_link
- removed link camera_right_ir_frame
- removed link camera_right_ir_optical_frame
- added link base_footprint
- link base_link: geometry visual box size=0.2 0.3 0.1
- link rear_left_wheel: geometry collision cylinder length=0.003 radius=0.077; visual cylinder length=0.003 radius=0.077
- link rear_right_wheel: geometry collision cylinder length=0.003 radius=0.077; visual cylinder length=0.003 radius=0.077
Joints:
- removed joint camera_color_joint
- removed joint camera_color_optical_joint
- removed joint camera_depth_joint
- removed joint camera_depth_optical_joint
- removed joint camera_joint
- removed joint camera_left_ir_joint
- removed joint camera_left_ir_optical_joint
- removed joint camera_link_joint
- removed joint camera_right_ir_joint
- removed joint camera_right_ir_optical_joint
- added joint base_joint: type fixed, parent base_footprint, child base_link, origin xyz=0 0 0 rpy=0 0 0
- joint front_left_wheel_joint: limit lower=-0.9 upper=0.9 effort=100 velocity=1 -> lower=-0.6 upper=0.6 effort=100 velocity=1; origin xyz=-0.061900000000000004 0.13175 0.107 rpy=1.5707963267948966 0 3.141592653589793 -> xyz=0.13175 -0.061900000000000004 0.107 rpy=0 0 3.141592653589793
- joint front_right_wheel_joint: limit lower=-0.9 upper=0.9 effort=100 velocity=1 -> lower=-0.6 upper=0.6 effort=100 velocity=1; origin xyz=-0.061900000000000004 -0.13175 0.107 rpy=1.5707963267948966 0 3.141592653589793 -> xyz=-0.13175 -0.061900000000000004 0.107 rpy=0 0 3.141592653589793

File: sim_ws/src/glide_robot/models/glide_description.urdf.xacro (robot description, xacro)
@@ -86,13 +86,13 @@
       <visual>
         <geometry>
-          <cylinder length="0.001" radius="0.001"/>
-        </geometry>
-        <origin rpy="0 0 0" xyz="0 0 0"/>
-        <material name="white"/>
-      </visual>
-      <collision>
-        <origin rpy="0 0 0" xyz="0 0 0"/>
-        <geometry>
-          <cylinder length="0.001" radius="0.001"/>
+          <cylinder length="${wheel_width}" radius="${wheel_radius}"/>
+        </geometry>
+        <origin rpy="0 0 0" xyz="0 0 0"/>
+        <material name="white"/>
+      </visual>
+      <collision>
+        <origin rpy="0 0 0" xyz="0 0 0"/>
+        <geometry>
+          <cylinder length="${wheel_width}" radius="${wheel_radius}"/>
         </geometry>
       </collision>
@@ -134,10 +134,11 @@
       <axis xyz="0 1 0"/>
     </joint> -->
+  <link name="base_footprint"/>
   <link name="base_link">
     <visual>
       <geometry>
-        <box size="${body_length} ${body_width} ${body_height}"/>
-      </geometry>
-      <origin rpy="0 0 0" xyz="0 0 ${body_center}"/>
+        <box size="${body_width} ${body_length} ${body_height}"/>
+      </geometry>
+      <origin rpy="0 0 1.57" xyz="0 0 ${body_center}"/>
       <material name="blue"/>
     </visual>
@@ -146,4 +147,9 @@
       <material>Gazebo/Blue</material>
   </gazebo>
+  <joint name="base_joint" type="fixed">
+      <origin rpy="0 0 0" xyz="0 0 0"/> <!-- 0 3.14 1.57-->
+      <child link="base_link"/>
+      <parent link="base_footprint"/>
+  </joint>
   <!-- <xacro:bar name="front" x_offset="${1.25*body_width}" z_offset="-${body_width}" parent_link="steer_bar_link"/> -->
   <xacro:steer_wheel name="right" offset="-0.1" xy_reflect="-1"/>
@@ -156,5 +162,5 @@
   <xacro:rotate_wheel name="right" offset="-0.1" xy_reflect="-1" />
   <xacro:rotate_wheel name="left" offset="-0.1" xy_reflect="1" />
-<link name="camera_bottom_screw_frame">
+<!-- <link name="camera_bottom_screw_frame">
     <visual>
       <geometry>
@@ -167,6 +173,6 @@
       </geometry>
     </collision>
-  </link>
-  <link name="camera_link"></link>
+  </link> -->
+  <!-- <link name="camera_link"></link>
   <link name="camera_depth_frame"></link>
   <link name="camera_depth_optical_frame"></link>
@@ -176,12 +182,12 @@
   <link name="camera_left_ir_optical_frame"></link>
   <link name="camera_right_ir_frame"></link>
-  <link name="camera_right_ir_optical_frame"></link>
-   <joint name="camera_joint" type="fixed">
+  <link name="camera_right_ir_optical_frame"></link> -->
+   <!-- <joint name="camera_joint" type="fixed">
     <parent link="base_link" />
     <child link="camera_bottom_screw_frame" />
     <pose xyz="0.4 0 0.25" rpy="0 0 0" />
-  </joint>
-  <joint name="camera_link_joint" type="fixed">
-    <parent link="camera_bottom_screw_frame" />
+  </joint> -->
+  <!-- <joint name="camera_link_joint" type="fixed">
+    <parent link="base_link" />
     <child link="camera_link" />
     <pose xyz="0 0.0175 0.0125 " rpy="0 0 0" />
@@ -226,5 +232,5 @@
     <child link="camera_right_ir_optical_frame" />
     <pose xyz="0 0 0 " rpy="-1.57 0 -1.57" />
-  </joint>
+  </joint> -->
   <link name="human_link">
     <visual>
